File: Schematic/MCU.sch (KiCad schematic (older format))
At the start: 37 parts, among them J1 Conn_ARM_JTAG_SWD_10, J2 Micro_SD_Card, SW1 SW_Push, SW2 SW_Push, U1 STM32F427VGTx, U2 AH1806-W, U3 FT232RL

Commit message: Continue work on layout
Connections:
- net FTDI_PWR_EN: now also U1.78 (PC10)
- net V1: now also R1.1, R2.1
- net V1_EN: now also U1.38 (PE7); no longer U1.66 (PC9)
- net VDD: no longer R1.1, R2.1
- net at U1.82 (PD1): now also R1.2, SW1.2
- net at U1.83 (PD2): now also R2.2, SW2.2
- no-connect marks 84 -> 81
Other:
- moved on the sheet: R1, SW1
Changed lines of the file:
@@
 Text HLabel 3900 4000 2    50   Input ~ 0
 FUEL_SCL
-Text HLabel 3500 6000 2    50   Input ~ 0
+Text HLabel 1600 4100 0    50   Input ~ 0
 V1_EN
 Text HLabel 3500 5900 2    50   Input ~ 0
@@
 L Switch:SW_Push SW1
 U 1 1 5E368629
-P 850 4350
-F 0 "SW1" V 896 4302 50  0000 R CNN
-F 1 "SW_Push" V 805 4302 50  0000 R CNN
-F 2 "Button_Switch_SMD:SW_Push_1P1T_NO_6x6mm_H9.5mm" H 850 4550 50  0001 C CNN
-F 3 "" H 850 4550 50  0001 C CNN
-	1    850  4350
+P 850 4450
+F 0 "SW1" V 896 4402 50  0000 R CNN
+F 1 "SW_Push" V 805 4402 50  0000 R CNN
+F 2 "Button_Switch_SMD:SW_Push_1P1T_NO_6x6mm_H9.5mm" H 850 4650 50  0001 C CNN
+F 3 "" H 850 4650 50  0001 C CNN
+	1    850  4450
 	0    -1   -1   0
 $EndComp
@@
 L Device:R R1
 U 1 1 5E368E6F
-P 850 4000
-F 0 "R1" H 920 4046 50  0000 L CNN
-F 1 "10K" H 920 3955 50  0000 L CNN
-F 2 "Resistor_SMD:R_0603_1608Metric_Pad1.05x0.95mm_HandSolder" V 780 4000 50  0001 C CNN
-F 3 "~" H 850 4000 50  0001 C CNN
-	1    850  4000
-	1    0    0    -1
-$EndComp
-Text HLabel 800  3750 0    50   Input ~ 0
-VDD
-Wire Wire Line
-	850  3850 850  3750
-Wire Wire Line
-	850  3750 800  3750
+P 850 4100
+F 0 "R1" H 920 4146 50  0000 L CNN
+F 1 "10K" H 920 4055 50  0000 L CNN
+F 2 "Resistor_SMD:R_0603_1608Metric_Pad1.05x0.95mm_HandSolder" V 780 4100 50  0001 C CNN
+F 3 "~" H 850 4100 50  0001 C CNN
+	1    850  4100
+	1    0    0    -1
+$EndComp
+Wire Wire Line
+	850  3950 850  3850
 $Comp
 L power:GND #PWR02
 U 1 1 5E36C004
-P 850 4550
-F 0 "#PWR02" H 850 4300 50  0001 C CNN
-F 1 "GND" H 855 4377 50  0000 C CNN
-F 2 "" H 850 4550 50  0001 C CNN
-F 3 "" H 850 4550 50  0001 C CNN
-	1    850  4550
+P 850 4650
+F 0 "#PWR02" H 850 4400 50  0001 C CNN
+F 1 "GND" H 855 4477 50  0000 C CNN
+F 2 "" H 850 4650 50  0001 C CNN
+F 3 "" H 850 4650 50  0001 C CNN
+	1    850  4650
 	1    0    0    -1
 $EndComp
@@
 	1    0    0    -1
 $EndComp
-Text HLabel 800  4900 0    50   Input ~ 0
-VDD
 Wire Wire Line
 	850  5000 850  4900
-Wire Wire Line
-	850  4900 800  4900
 $Comp
 L power:GND #PWR03
@@
 NoConn ~ 3500 5700
 NoConn ~ 3500 5800
-NoConn ~ 3500 6100
 NoConn ~ 3500 6200
 NoConn ~ 3500 6300
@@
 NoConn ~ 1700 5500
 NoConn ~ 1700 5400
-NoConn ~ 1700 5300
-NoConn ~ 1700 5200
 NoConn ~ 1700 5100
 NoConn ~ 1700 4900
@@
 NoConn ~ 1700 4300
 NoConn ~ 1700 4200
-NoConn ~ 1700 4100
+NoConn ~ 3500 6000
 NoConn ~ 1700 4000
 NoConn ~ 1700 3900
@@
 	4800 1050 5250 1050
 Connection ~ 4800 1050
+Wire Wire Line
+	1700 4100 1600 4100
+Text HLabel 750  4900 0    50   Input ~ 0
+V1
+Wire Wire Line
+	850  4900 750  4900
+Text HLabel 700  3850 0    50   Input ~ 0
+V1
+Wire Wire Line
+	700  3850 850  3850
+Wire Wire Line
+	850  5300 1700 5300
+Connection ~ 850  5300
+Wire Wire Line
+	1700 5200 1400 5200
+Wire Wire Line
+	1400 5200 1400 4250
+Wire Wire Line
+	1400 4250 850  4250
+Connection ~ 850  4250
+Text Label 3600 6100 0    50   ~ 0
+FTDI_PWR_EN
+Wire Wire Line
+	3600 6100 3500 6100
 $EndSCHEMATC

Commit message: Rev 0 historical data
Parts:
- J1: symbol Connector:Conn_ARM_JTAG_SWD_10 -> SoundBoard-rescue:Conn_ARM_JTAG_SWD_10-Connector
- J2: symbol Connector:Micro_SD_Card -> SoundBoard-rescue:Micro_SD_Card-Connector
Changed lines of the file:
@@
 EESchema Schematic File Version 4
-EELAYER 30 0
+LIBS:SoundBoard-cache
+EELAYER 26 0
 EELAYER END
 $Descr A4 11693 8268
@@
 Connection ~ 2400 1400
 $Comp
-L Connector:Micro_SD_Card J2
+L SoundBoard-rescue:Micro_SD_Card-Connector J2
 U 1 1 5E2EDD03
 P 5800 6000
@@
 NRESET
 $Comp
-L Connector:Conn_ARM_JTAG_SWD_10 J1
+L SoundBoard-rescue:Conn_ARM_JTAG_SWD_10-Connector J1
 U 1 1 5E2FC7AF
 P 4900 3000
+AR Path="/5E2FC7AF" Ref="J1"  Part="1"
+AR Path="/5E238EA5/5E2FC7AF" Ref="J1"  Part="1"
 F 0 "J1" H 4450 3500 50  0000 R CNN
 F 1 "Conn_ARM_JTAG_SWD_10" H 4850 3600 50  0000 R CNN
