File: Schematic/SoundBoard.sch (KiCad schematic (older format))
At the start: 0 parts

Commit message: Add passives
Changed lines of the file:
@@
 F0 "MCU" 50
 F1 "MCU.sch" 50
+F2 "VDD" I R 2200 1250 50
+F3 "AUDIO_FROM_DAC" I L 1150 1850 50
+F4 "V1" I R 2200 1900 50
+F5 "FUEL_SDA" I R 2200 1450 50
+F6 "FUEL_SCL" I R 2200 1550 50
+F7 "V1_EN" I R 2200 1350 50
+F8 "SHUTDOWN_AMP" I L 1150 1950 50
+F9 "USB_P" I R 2200 1650 50
+F10 "USB_N" I R 2200 1750 50
 $EndSheet
 $Sheet
@@
 F0 "Audio" 50
 F1 "Audio.sch" 50
-F2 "SHUTDOWN" I R 2200 2300 50
-F3 "AUDIO_FROM_DAC" I R 2200 2400 50
+F2 "SHUTDOWN" I L 1150 2300 50
+F3 "AUDIO_FROM_DAC" I L 1150 2400 50
 F4 "V1" I R 2200 2550 50
 $EndSheet
@@
 F5 "FUEL_SDA" I L 2750 1450 50
 F6 "FUEL_SCL" I L 2750 1550 50
+F7 "USB_P" I L 2750 1650 50
+F8 "USB_N" I L 2750 1750 50
 $EndSheet
 Wire Wire Line
@@
 Wire Wire Line
 	2550 1900 2750 1900
+Wire Wire Line
+	2200 1250 2750 1250
+Wire Wire Line
+	2200 1450 2750 1450
+Wire Wire Line
+	2200 1550 2750 1550
+Wire Wire Line
+	2200 1900 2550 1900
+Connection ~ 2550 1900
+Wire Wire Line
+	2200 1350 2750 1350
+Wire Wire Line
+	1150 2300 1100 2300
+Wire Wire Line
+	1100 2300 1100 1950
+Wire Wire Line
+	1150 1950 1100 1950
+Wire Wire Line
+	1150 2400 1050 2400
+Wire Wire Line
+	1050 2400 1050 1850
+Wire Wire Line
+	1050 1850 1150 1850
+Wire Wire Line
+	2200 1650 2750 1650
+Wire Wire Line
+	2200 1750 2750 1750
 $EndSCHEMATC
