File: Schematic/Soundboard/Audio.sch (KiCad schematic (older format))
At the start: 0 parts

Commit message: Begin rev 2 part selection and schematic
Parts:
- added C5, C6, C7, C8, C9: C, Capacitor_SMD:C_0603_1608Metric_Pad1.05x0.95mm_HandSolder, symbol Device:C
- added J4: AudioJack3, Connector_Audio:Jack_3.5mm_CUI_SJ-3523-SMT_Horizontal, symbol Connector:AudioJack3
- added U5: CS4334, Package_SO:SOIC-8-N7_3.9x4.9mm_P1.27mm, symbol Soundboard:CS4334
- added U6: LM4811, Package_SO:TSSOP-10_3x3mm_P0.5mm, symbol Amplifier_Audio:LM4811
Connections:
- net labels added: +5V, GND
- wire segments 0 -> 15
Changed lines of the file:
@@
 $Descr A4 11693 8268
 encoding utf-8
-Sheet 1 4
+Sheet 3 6
 Title ""
 Date ""
@@
 Comment4 ""
 $EndDescr
+$Comp
+L Amplifier_Audio:LM4811 U6
+U 1 1 5F2C1ECA
+P 5250 3550
+F 0 "U6" H 5500 4150 50  0000 C CNN
+F 1 "LM4811" H 5500 4050 50  0000 C CNN
+F 2 "Package_SO:TSSOP-10_3x3mm_P0.5mm" H 5250 3550 50  0001 C CIN
+F 3 "http://www.ti.com/lit/ds/symlink/lm4811.pdf" H 5250 3550 50  0001 C CNN
+	1    5250 3550
+	1    0    0    -1
+$EndComp
+$Comp
+L Connector:AudioJack3 J4
+U 1 1 5F2C4721
+P 6850 3450
+F 0 "J4" H 6570 3383 50  0000 R CNN
+F 1 "AudioJack3" H 6570 3474 50  0000 R CNN
+F 2 "Connector_Audio:Jack_3.5mm_CUI_SJ-3523-SMT_Horizontal" H 6850 3450 50  0001 C CNN
+F 3 "~" H 6850 3450 50  0001 C CNN
+	1    6850 3450
+	-1   0    0    1
+$EndComp
+$Comp
+L Device:C C8
+U 1 1 5F2C5DF4
+P 6050 3350
+F 0 "C8" V 5798 3350 50  0000 C CNN
+F 1 "C" V 5889 3350 50  0000 C CNN
+F 2 "Capacitor_SMD:C_0603_1608Metric_Pad1.05x0.95mm_HandSolder" H 6088 3200 50  0001 C CNN
+F 3 "~" H 6050 3350 50  0001 C CNN
+	1    6050 3350
+	0    1    1    0
+$EndComp
+$Comp
+L Device:C C9
+U 1 1 5F2C644C
+P 6050 3550
+F 0 "C9" V 6200 3650 50  0000 C CNN
+F 1 "C" V 6200 3550 50  0000 C CNN
+F 2 "Capacitor_SMD:C_0603_1608Metric_Pad1.05x0.95mm_HandSolder" H 6088 3400 50  0001 C CNN
+F 3 "~" H 6050 3550 50  0001 C CNN
+	1    6050 3550
+	0    1    1    0
+$EndComp
+Wire Wire Line
+	5650 3350 5900 3350
+Wire Wire Line
+	6200 3350 6650 3350
+Wire Wire Line
+	5650 3550 5900 3550
+Wire Wire Line
+	6200 3550 6200 3450
+Wire Wire Line
+	6200 3450 6650 3450
+$Comp
+L power:GND #PWR0116
+U 1 1 5F2C9761
+P 6600 3550
+F 0 "#PWR0116" H 6600 3300 50  0001 C CNN
+F 1 "GND" H 6605 3377 50  0000 C CNN
+F 2 "" H 6600 3550 50  0001 C CNN
+F 3 "" H 6600 3550 50  0001 C CNN
+	1    6600 3550
+	1    0    0    -1
+$EndComp
+Wire Wire Line
+	6600 3550 6650 3550
+$Comp
+L Device:C C7
+U 1 1 5F2CA65B
+P 5750 3900
+F 0 "C7" H 5865 3946 50  0000 L CNN
+F 1 "C" H 5865 3855 50  0000 L CNN
+F 2 "Capacitor_SMD:C_0603_1608Metric_Pad1.05x0.95mm_HandSolder" H 5788 3750 50  0001 C CNN
+F 3 "~" H 5750 3900 50  0001 C CNN
+	1    5750 3900
+	1    0    0    -1
+$EndComp
+Wire Wire Line
+	5750 3750 5650 3750
+$Comp
+L power:GND #PWR0117
+U 1 1 5F2CAC1B
+P 5750 4050
+F 0 "#PWR0117" H 5750 3800 50  0001 C CNN
+F 1 "GND" H 5755 3877 50  0000 C CNN
+F 2 "" H 5750 4050 50  0001 C CNN
+F 3 "" H 5750 4050 50  0001 C CNN
+	1    5750 4050
+	1    0    0    -1
+$EndComp
+$Comp
+L power:GND #PWR0118
+U 1 1 5F2CB1F7
+P 5250 4050
+F 0 "#PWR0118" H 5250 3800 50  0001 C CNN
+F 1 "GND" H 5255 3877 50  0000 C CNN
+F 2 "" H 5250 4050 50  0001 C CNN
+F 3 "" H 5250 4050 50  0001 C CNN
+	1    5250 4050
+	1    0    0    -1
+$EndComp
+$Comp
+L Device:C C5
+U 1 1 5F2CBAC4
+P 4700 3350
+F 0 "C5" V 4448 3350 50  0000 C CNN
+F 1 "C" V 4539 3350 50  0000 C CNN
+F 2 "Capacitor_SMD:C_0603_1608Metric_Pad1.05x0.95mm_HandSolder" H 4738 3200 50  0001 C CNN
+F 3 "~" H 4700 3350 50  0001 C CNN
+	1    4700 3350
+	0    1    1    0
+$EndComp
+$Comp
+L Device:C C6
+U 1 1 5F2CC435
+P 4700 3550
+F 0 "C6" V 4600 3400 50  0000 C CNN
+F 1 "C" V 4600 3300 50  0000 C CNN
+F 2 "Capacitor_SMD:C_0603_1608Metric_Pad1.05x0.95mm_HandSolder" H 4738 3400 50  0001 C CNN
+F 3 "~" H 4700 3550 50  0001 C CNN
+	1    4700 3550
+	0    1    1    0
+$EndComp
+$Comp
+L Soundboard:CS4334 U5
+U 1 1 5F2D3B6C
+P 3650 3150
+F 0 "U5" H 3650 3265 50  0000 C CNN
+F 1 "CS4334" H 3650 3174 50  0000 C CNN
+F 2 "Package_SO:SOIC-8-N7_3.9x4.9mm_P1.27mm" H 3650 3150 50  0001 C CNN
+F 3 "" H 3650 3150 50  0001 C CNN
+	1    3650 3150
+	1    0    0    -1
+$EndComp
+Wire Wire Line
+	4050 3400 4400 3400
+Wire Wire Line
+	4400 3400 4400 3350
+Wire Wire Line
+	4400 3350 4550 3350
+Wire Wire Line
+	4050 3500 4400 3500
+Wire Wire Line
+	4400 3500 4400 3550
+Wire Wire Line
+	4400 3550 4550 3550
+$Comp
+L power:GND #PWR0119
+U 1 1 5F2DD9C3
+P 4150 3600
+F 0 "#PWR0119" H 4150 3350 50  0001 C CNN
+F 1 "GND" H 4155 3427 50  0000 C CNN
+F 2 "" H 4150 3600 50  0001 C CNN
+F 3 "" H 4150 3600 50  0001 C CNN
+	1    4150 3600
+	1    0    0    -1
+$EndComp
+Wire Wire Line
+	4150 3600 4050 3600
+$Comp
+L power:+5V #PWR0120
+U 1 1 5F2DE266
+P 4150 3300
+F 0 "#PWR0120" H 4150 3150 50  0001 C CNN
+F 1 "+5V" H 4165 3473 50  0000 C CNN
+F 2 "" H 4150 3300 50  0001 C CNN
+F 3 "" H 4150 3300 50  0001 C CNN
+	1    4150 3300
+	1    0    0    -1
+$EndComp
+Wire Wire Line
+	4150 3300 4050 3300
+$Comp
+L power:+5V #PWR0121
+U 1 1 5F2E070A
+P 5250 3050
+F 0 "#PWR0121" H 5250 2900 50  0001 C CNN
+F 1 "+5V" H 5265 3223 50  0000 C CNN
+F 2 "" H 5250 3050 50  0001 C CNN
+F 3 "" H 5250 3050 50  0001 C CNN
+	1    5250 3050
+	1    0    0    -1
+$EndComp
 $EndSCHEMATC
