File: Schematic/Soundboard/Microcontroller.sch (KiCad schematic (older format))
At the start: 0 parts

Commit message: Begin rev 2 part selection and schematic
Parts:
- added C1, C2, C3, C4: C, Capacitor_SMD:C_0603_1608Metric_Pad1.05x0.95mm_HandSolder, symbol Device:C
- added D?: LED, symbol Device:LED
- added J1: USB_B_Micro, Connector_USB:USB_Micro-B_Amphenol_10103594-0001LF_Horizontal, symbol Connector:USB_B_Micro
- added J2: Conn_ARM_JTAG_SWD_10, Connector_PinHeader_1.27mm:PinHeader_2x05_P1.27mm_Vertical, symbol Connector:Conn_ARM_JTAG_SWD_10
- added J3: Micro_SD_Card, Connector_Card:microSD_HC_Hirose_DM3D-SF, symbol Connector:Micro_SD_Card
- added J?: Conn_02x02_Counter_Clockwise, symbol Connector_Generic:Conn_02x02_Counter_Clockwise
- added R?: R, symbol Device:R
- added U1: STM32f429IIT6-units, Package_QFP:LQFP-176_24x24mm_P0.5mm, symbol Soundboard:STM32f429IIT6-units
- added U2: USBLC6-4SC6, Package_TO_SOT_SMD:SOT-23-6, symbol Power_Protection:USBLC6-4SC6
- added U3: W25Q128JVS, Package_SO:SOIC-8_5.23x5.23mm_P1.27mm, symbol Memory_Flash:W25Q128JVS
- added U4: BMI160, Package_LGA:Bosch_LGA-14_3x2.5mm_P0.5mm, symbol Sensor_Motion:BMI160
Connections:
- new net: D?.1 (K), R?.1
- new net +1V8: C3.1, C4.1
- new net +3V3: C1.1, C2.1, J3.4 (VDD), J?.1 (Pin_1), U3.8 (VCC), U4.5 (VDDIO), U4.8 (VDD)
- new net FLASH_CS: U3.1 (~CS)
- new net GND: C1.2, C2.2, C3.2, C4.2, J1.5 (GND), J1.6 (Shield), J2.3 (GND), J2.5 (GND), J2.9 (GNDDetect), J3.6 (VSS), J3.9 (SHIELD), J?.2 (Pin_2), R?.2, U2.2 (GND), U3.4 (GND), U4.6 (GNDIO), U4.7 (GND)
- new net IMU_CS: U4.12 (CSB)
- new net NRST: J2.10 (~RESET~)
- new net SCL: J?.3 (Pin_3)
- new net SDA: J?.4 (Pin_4)
- new net SDIO_CK: J3.5 (CLK)
- new net SDIO_CMD: J3.3 (CMD)
- new net SDIO_D0: J3.7 (DAT0)
- new net SDIO_D1: J3.8 (DAT1)
- new net SDIO_D2: J3.1 (DAT2)
- new net SDIO_D3: J3.2 (DAT3/CD)
- new net SPI_MISO: U3.2 (DO(IO1)), U4.1 (SDO)
- new net SPI_MOSI: U3.5 (DI(IO0)), U4.14 (SDx)
- new net SPI_SCLK: U3.6 (CLK), U4.13 (SCx)
- new net SWCLK: J2.4 (SWDCLK/TCK)
- new net SWDIO: J2.2 (SWDIO/TMS)
- new net SWO: J2.6 (SWO/TDO)
- new net USBD_N: J1.2 (D-), U2.3 (I/O2)
- new net USBD_P: J1.3 (D+), U2.1 (I/O1)
- new net VDD: J2.1 (VTref)
- new net V_USB_5: J1.1 (VBUS), U2.5 (VBUS)
- no-connect marks 0 -> 10
