File: Schematic/Soundboard/Power.sch (KiCad schematic (older format))
At the start: 0 parts

Commit message: Begin rev 2 part selection and schematic
Parts:
- added C10, C11: 2.2u, Capacitor_SMD:C_0603_1608Metric_Pad1.05x0.95mm_HandSolder, symbol Device:C
- added C? (x16): 100n, symbol Device:C
- added C?: 4.7u, symbol Device:C
- added C? (x2): 1u, symbol Device:C
- added C?: 10n, symbol Device:C
- added D? (x2): D_Schottky, symbol Device:D_Schottky
- added D? (x2): LED, symbol Device:LED
- added J?: Conn_01x02, symbol Connector_Generic:Conn_01x02
- added R? (x3): R, symbol Device:R
- added R?: 0, symbol Device:R
- added U1: STM32f429IIT6-units, Package_QFP:LQFP-176_24x24mm_P0.5mm, symbol Soundboard:STM32f429IIT6-units
- added U?: MIC5504-3.3YM5, Package_TO_SOT_SMD:SOT-23-5, symbol Regulator_Linear:MIC5504-3.3YM5
- added U?: MCP73831-2-OT, Package_TO_SOT_SMD:SOT-23-5, symbol Battery_Management:MCP73831-2-OT
Connections:
- new net: C?.1, C?.1, U1.38 (VREF+)
- new net: U1.102 (VSS), U1.113 (VSS), U1.126 (VSS), U1.135 (VSS), U1.14 (VSS), U1.148 (VSS), U1.158 (VSS), U1.22 (VSS), U1.61 (VSS), U1.71 (VSS), U1.90 (VSS)
- new net: C10.1, U1.125 (VCAP_2)
- new net: R?.1, U1.6 (VBAT)
- new net: C11.1, U1.81 (VCAP_1)
- new net: D?.1 (K), R?.1
- new net: R?.1, U?.1 (STAT)
- new net: R?.1, U?.5 (PROG)
- new net: D?.1 (K), R?.2
- new net GND: C10.2, C11.2, C?.2, C?.2, C?.2, C?.2, C?.2, C?.2, C?.2, C?.2, C?.2, C?.2, C?.2, C?.2, C?.2, C?.2, C?.2, C?.2, C?.2, C?.2, C?.2, C?.2, J?.2 (Pin_2), R?.2, R?.2, U1.37 (VSSA), U?.2 (GND), U?.2 (VSS)
- new net V_BAT: D?.2 (A), J?.1 (Pin_1), R?.2, U?.3 (VBAT)
- new net V_INT: D?.1 (K), D?.1 (K), U?.1 (VIN), U?.3 (EN)
- new net V_MCU: C?.1, C?.1, C?.1, C?.1, C?.1, C?.1, C?.1, C?.1, C?.1, C?.1, C?.1, C?.1, C?.1, C?.1, C?.1, C?.1, C?.1, C?.1, D?.2 (A), U1.103 (VDD), U1.114 (VDD), U1.127 (VDD), U1.136 (VDD), U1.149 (VDD), U1.15 (VDD), U1.159 (VDD), U1.172 (VDD), U1.23 (VDD), U1.36 (VDD), U1.39 (VDDA), U1.49 (VDD), U1.62 (VDD), U1.72 (VDD), U1.82 (VDD), U1.91 (VDD), U?.5 (VOUT)
- new net V_USB_5: D?.2 (A), D?.2 (A), U?.4 (VDD)
Other:
- note added: "LIPO Battery\n"
- note added: "LIPO Charger\n"
